File: Pot.butt_pcb/Pot.butt_pcb/dcdc_convs.kicad_sch (KiCad schematic)
At the start: 29 parts, among them U3 LMR62421XMF, U4 LMR62421XMF

Commit message: main_func pcb done
Parts:
- C62, C63: value 10u -> 10uF
- C64: value 10n -> 10nF
- C65: value 100n -> 100nF
Changed lines of the file:
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@@
       (effects (font (size 1.27 1.27)) (justify left))
     )
-    (property "Value" "10u" (id 1) (at 199.39 113.0299 0)
+    (property "Value" "10uF" (id 1) (at 199.39 113.0299 0)
       (effects (font (size 1.27 1.27)) (justify left))
     )
@@
       (effects (font (size 1.27 1.27)) (justify left))
     )
-    (property "Value" "100n" (id 1) (at 250.19 113.0299 0)
+    (property "Value" "100nF" (id 1) (at 250.19 113.0299 0)
       (effects (font (size 1.27 1.27)) (justify left))
     )
@@
       (effects (font (size 1.27 1.27)) (justify left))
     )
-    (property "Value" "10u" (id 1) (at 226.06 113.0299 0)
+    (property "Value" "10uF" (id 1) (at 226.06 113.0299 0)
       (effects (font (size 1.27 1.27)) (justify left))
     )
@@
       (effects (font (size 1.27 1.27)) (justify left))
     )
-    (property "Value" "10n" (id 1) (at 238.76 113.0299 0)
-      (effects (font (size 1.27 1.27)) (justify left))
-    )
+    (property "Value" "10nF" (id 1) (at 238.76 113.0299 0)
+      (effects (font (size 1.27 1.27)) (justify left))
+    )
