File: Pot.butt_pcb/Pot.butt_pcb/Switches.kicad_sch (KiCad schematic)
At the start: 16 parts, among them SW2 SW_DPDT, SW3 SW_DPDT, SW4 SW_DPDT, SW5 SW_DPDT, SW6 SW_DPDT, SW7 SW_DPDT, SW8 SW_DPDT, SW9 SW_DPDT

Commit message: Pot.but_pcb in progress
Parts:
- SW2, SW3, SW4, SW5, SW6, SW7, SW8, SW9: footprint Connector_PinHeader_2.54mm:PinHeader_1x03_P2.54mm_Horizontal -> Connector_PinSocket_2.54mm:PinSocket_1x03_P2.54mm_Vertical
Changed lines of the file:
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@@
     (property "Reference" "SW7" (id 0) (at 180.34 91.44 0))
     (property "Value" "SW_DPDT" (id 1) (at 180.34 93.98 0))
-    (property "Footprint" "Connector_PinHeader_2.54mm:PinHeader_1x03_P2.54mm_Horizontal" (id 2) (at 180.34 99.06 0)
+    (property "Footprint" "Connector_PinSocket_2.54mm:PinSocket_1x03_P2.54mm_Vertical" (id 2) (at 180.34 99.06 0)
       (effects (font (size 1.27 1.27)) hide)
     )
@@
     (property "Reference" "SW4" (id 0) (at 129.54 40.64 0))
     (property "Value" "SW_DPDT" (id 1) (at 129.54 43.18 0))
-    (property "Footprint" "Connector_PinHeader_2.54mm:PinHeader_1x03_P2.54mm_Horizontal" (id 2) (at 129.54 48.26 0)
+    (property "Footprint" "Connector_PinSocket_2.54mm:PinSocket_1x03_P2.54mm_Vertical" (id 2) (at 129.54 48.26 0)
       (effects (font (size 1.27 1.27)) hide)
     )
@@
     (property "Reference" "SW8" (id 0) (at 231.14 40.64 0))
     (property "Value" "SW_DPDT" (id 1) (at 231.14 43.18 0))
-    (property "Footprint" "Connector_PinHeader_2.54mm:PinHeader_1x03_P2.54mm_Horizontal" (id 2) (at 231.14 48.26 0)
+    (property "Footprint" "Connector_PinSocket_2.54mm:PinSocket_1x03_P2.54mm_Vertical" (id 2) (at 231.14 48.26 0)
       (effects (font (size 1.27 1.27)) hide)
     )
@@
     (property "Reference" "SW6" (id 0) (at 180.34 40.64 0))
     (property "Value" "SW_DPDT" (id 1) (at 180.34 43.18 0))
-    (property "Footprint" "Connector_PinHeader_2.54mm:PinHeader_1x03_P2.54mm_Horizontal" (id 2) (at 180.34 48.26 0)
+    (property "Footprint" "Connector_PinSocket_2.54mm:PinSocket_1x03_P2.54mm_Vertical" (id 2) (at 180.34 48.26 0)
       (effects (font (size 1.27 1.27)) hide)
     )
@@
     (property "Reference" "SW5" (id 0) (at 129.54 91.44 0))
     (property "Value" "SW_DPDT" (id 1) (at 129.54 93.98 0))
-    (property "Footprint" "Connector_PinHeader_2.54mm:PinHeader_1x03_P2.54mm_Horizontal" (id 2) (at 129.54 99.06 0)
+    (property "Footprint" "Connector_PinSocket_2.54mm:PinSocket_1x03_P2.54mm_Vertical" (id 2) (at 129.54 99.06 0)
       (effects (font (size 1.27 1.27)) hide)
     )
@@
     (property "Reference" "SW9" (id 0) (at 231.14 91.44 0))
     (property "Value" "SW_DPDT" (id 1) (at 231.14 93.98 0))
-    (property "Footprint" "Connector_PinHeader_2.54mm:PinHeader_1x03_P2.54mm_Horizontal" (id 2) (at 231.14 99.06 0)
+    (property "Footprint" "Connector_PinSocket_2.54mm:PinSocket_1x03_P2.54mm_Vertical" (id 2) (at 231.14 99.06 0)
       (effects (font (size 1.27 1.27)) hide)
     )
@@
     (property "Reference" "SW3" (id 0) (at 66.04 91.44 0))
     (property "Value" "SW_DPDT" (id 1) (at 66.04 93.98 0))
-    (property "Footprint" "Connector_PinHeader_2.54mm:PinHeader_1x03_P2.54mm_Horizontal" (id 2) (at 66.04 99.06 0)
+    (property "Footprint" "Connector_PinSocket_2.54mm:PinSocket_1x03_P2.54mm_Vertical" (id 2) (at 66.04 99.06 0)
       (effects (font (size 1.27 1.27)) hide)
     )
@@
     (property "Reference" "SW2" (id 0) (at 66.04 40.64 0))
     (property "Value" "SW_DPDT" (id 1) (at 66.04 43.18 0))
-    (property "Footprint" "Connector_PinHeader_2.54mm:PinHeader_1x03_P2.54mm_Horizontal" (id 2) (at 66.04 48.26 0)
-      (effects (font (size 1.27 1.27)) hide)
-    )
+    (property "Footprint" "Connector_PinSocket_2.54mm:PinSocket_1x03_P2.54mm_Vertical" (id 2) (at 66.04 48.26 0)
+      (effects (font (size 1.27 1.27)) hide)
+    )

Commit message: pcb design fixing
Parts:
- removed R1, R2, R3, R4, R5, R6, R7, R8: 100, Resistor_SMD:R_0805_2012Metric_Pad1.20x1.40mm_HandSolder, symbol Device:R
- removed SW2, SW3, SW4, SW5, SW6, SW7, SW8, SW9: SW_DPDT, Connector_PinSocket_2.54mm:PinSocket_1x03_P2.54mm_Vertical, symbol Switch:SW_DPDT_x2
