File: Pot.butt_pcb/Pot.butt_pcb/Pot.butt_pcb.kicad_pcb (KiCad board)
At the start: 2 copper layers, 220 x 142 mm, 195 parts, among them J1 Conn_01x10_Male, J2 Conn_01x05_Male, J3 Conn_01x05_Male, J4 Conn_01x40_Male, J5 Conn_01x40_Male, J6 Conn_01x40_Male, SW1 SW_Push, SW10 SW_Push, SW11 Cherry_MX_1u, SW12 Cherry_MX_1u, SW13 Cherry_MX_1u, SW14 Cherry_MX_1u, SW15 Cherry_MX_1u, SW16 Cherry_MX_1u, SW17 Cherry_MX_1u, SW18 Cherry_MX_1u, SW19 Cherry_MX_1u, SW20 Cherry_MX_1u, SW21 Cherry_MX_1u, SW22 Cherry_MX_1u, SW23 Cherry_MX_1u, SW24 Cherry_MX_1u, SW25 Cherry_MX_1u, SW26 Cherry_MX_1u, SW27 Cherry_MX_1u, SW28 Cherry_MX_1u, SW29 Cherry_MX_1u, SW30 Cherry_MX_1u, SW31 Cherry_MX_1u, SW32 Cherry_MX_1u, SW33 Cherry_MX_1u, SW34 Cherry_MX_1u, SW35 Cherry_MX_1u, U1 STM32G030K6T6, U2 STM32G030K6T6, U3 LMR62421XMF, U4 LMR62421XMF

Commit message: gerber files generated
Parts:
- removed REF** (x6): MountingHole_3.2mm_M3_Pad_Via, MountingHole:MountingHole_3.2mm_M3_Pad_Via
- added H1: MountingHole, MountingHole:MountingHole_3.2mm_M3_Pad_Via, F.Cu at (69.0, 28.0)
- added H2: MountingHole, MountingHole:MountingHole_3.2mm_M3_Pad_Via, F.Cu at (198.0, 28.0)
- added H3: MountingHole, MountingHole:MountingHole_3.2mm_M3_Pad_Via, F.Cu at (247.0, 28.0)
- added H4: MountingHole, MountingHole:MountingHole_3.2mm_M3_Pad_Via, F.Cu at (240.0, 160.0)
- added H5: MountingHole, MountingHole:MountingHole_3.2mm_M3_Pad_Via, F.Cu at (198.0, 160.0)
- added H6: MountingHole, MountingHole:MountingHole_3.2mm_M3_Pad_Via, F.Cu at (69.0, 160.0)
- J4, J5, J6: moved to B.Cu
- moved J4 48.3 mm to (56.7, 85.3)
- moved J5 48.3 mm to (56.9, 151.3)
- moved J6 48.3 mm to (128.3, 145.9)
Connections:
- J4 pad 10: 3.3VA -> ADC_in7s
- J4 pad 12: ADC_in2s -> 3.3VA
- J4 pad 14: 3.3VA -> ADC_in6s
- J4 pad 16: ADC_in3s -> 3.3VA
- J4 pad 18: 3.3VA -> ADC_in5s
- J4 pad 2: 3.3VA -> ADC_in1p
- J4 pad 20: ADC_in4s -> 3.3VA
- J4 pad 22: 3.3VA -> ADC_in4s
- J4 pad 24: ADC_in5s -> 3.3VA
- J4 pad 26: 3.3VA -> ADC_in3s
- J4 pad 28: ADC_in6s -> 3.3VA
- J4 pad 30: 3.3VA -> ADC_in2s
- J4 pad 32: ADC_in7s -> 3.3VA
- J4 pad 34: 3.3VA -> ADC_in1s
- J4 pad 36: ADC_in0p -> 3.3VA
- J4 pad 38: 3.3VA -> ADC_in0s
- J4 pad 4: ADC_in0s -> 3.3VA
- J4 pad 40: ADC_in1p -> 3.3VA
- J4 pad 6: 3.3VA -> ADC_in0p
- J4 pad 8: ADC_in1s -> 3.3VA
- J5 pad 10: 3.3VA -> ADC_in9p
- J5 pad 12: ADC_in4p -> 3.3VA
- J5 pad 14: 3.3VA -> ADC_in8p
- J5 pad 16: ADC_in5p -> 3.3VA
- J5 pad 18: 3.3VA -> ADC_in7p
- J5 pad 2: 3.3VA -> ADC_in11p
- J5 pad 20: ADC_in6p -> 3.3VA
- J5 pad 22: 3.3VA -> ADC_in6p
- J5 pad 24: ADC_in7p -> 3.3VA
- J5 pad 26: 3.3VA -> ADC_in5p
- J5 pad 28: ADC_in8p -> 3.3VA
- J5 pad 30: 3.3VA -> ADC_in4p
- J5 pad 32: ADC_in9p -> 3.3VA
- J5 pad 34: 3.3VA -> ADC_in3p
- J5 pad 36: ADC_in10p -> 3.3VA
- J5 pad 38: 3.3VA -> ADC_in2p
- J5 pad 4: ADC_in2p -> 3.3VA
- J5 pad 40: ADC_in11p -> 3.3VA
- J5 pad 6: 3.3VA -> ADC_in10p
- J5 pad 8: ADC_in3p -> 3.3VA
- J6 pad 10: +3V3 -> SW8
- J6 pad 12: SW3 -> +3V3
- J6 pad 14: +3V3 -> SW7
- J6 pad 16: SW4 -> +3V3
- J6 pad 18: +3V3 -> SW6
- J6 pad 2: +3V3 -> GND
- J6 pad 20: SW5 -> +3V3
- J6 pad 22: +3V3 -> SW5
- J6 pad 24: SW6 -> +3V3
- J6 pad 26: +3V3 -> SW4
- J6 pad 28: SW7 -> +3V3
- J6 pad 30: +3V3 -> SW3
- J6 pad 32: SW8 -> +3V3
- J6 pad 34: GND -> SW2
- J6 pad 36: GND -> +3V3
- J6 pad 38: GND -> SW1
- J6 pad 4: SW1 -> GND
- J6 pad 40: GND -> +3V3
- J6 pad 6: +3V3 -> GND
- J6 pad 8: SW2 -> GND
Routing:
- net GND: vias 1013 -> 1015
- net (no net): vias 4 -> 0
