File: Pot.butt_pcb/Pot.butt_pcb/Pot.butt_pcb.kicad_sch (KiCad schematic)
At the start: 0 parts

Commit message: fixing keyboard and pot project schematics
Other:
- added sheet dcdc_convs (dcdc_convs.kicad_sch)

Commit message: pcb design fixing
Other:
- sheet slide_potentiometer renamed potentiometer_switches
- removed sheet Switches
- removed sheet plugin_potentiometer
