File: main_func/main_func/midi_jacks.kicad_sch (KiCad schematic)
At the start: 18 parts, among them J4 Korean Hroparts Elec PJ-3250-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, J8 Conn_01x02_Male, U10 MIDI_THRU, U11 SN74HCT04DR, U5 6N137, U8 MIDI_OUT, U9 MIDI_IN

Commit message: pcb design fixing
Parts:
- removed J8: Conn_01x02_Male, Capacitor_THT:C_Rect_L7.5mm_W6.5mm_P5.00mm, symbol Connector:Conn_01x02_Male
- added J6: Conn_01x04_Male, Connector_PinHeader_2.54mm:PinHeader_1x04_P2.54mm_Vertical, symbol Connector:Conn_01x04_Male
Connections:
- net GND: now also J6.1 (Pin_1), J6.3 (Pin_3); no longer U9.2, U9.6
- net SOUTL: now also J6.2 (Pin_2)
- net SOUTR: now also J6.4 (Pin_4)
- new net MIDI_IN_GND: U9.2, U9.6
Changed lines of the file:
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@@
 (kicad_sch (version 20211123) (generator eeschema)
   (paper "A4")
+  (junction (at 63.5 35.56) (diameter 0) (color 0 0 0 0)
+  )
   (junction (at 214.63 53.34) (diameter 0) (color 0 0 0 0)
   )
@@
   (junction (at 259.08 50.8) (diameter 0) (color 0 0 0 0)
   )
+  (junction (at 184.15 132.08) (diameter 0) (color 0 0 0 0)
+  )
   (wire (pts (xy 171.45 59.69) (xy 171.45 60.96))
     (stroke (width 0) (type default) (color 0 0 0 0))
   )
-  (wire (pts (xy 72.39 30.48) (xy 72.39 33.02))
+  (wire (pts (xy 72.39 30.48) (xy 72.39 35.56))
     (stroke (width 0) (type default) (color 0 0 0 0))
   )
@@
     (stroke (width 0) (type default) (color 0 0 0 0))
   )
+  (wire (pts (xy 184.15 132.08) (xy 184.15 127))
+    (stroke (width 0) (type default) (color 0 0 0 0))
+  )
   (wire (pts (xy 171.45 52.07) (xy 171.45 50.8))
     (stroke (width 0) (type default) (color 0 0 0 0))
@@
     (stroke (width 0) (type default) (color 0 0 0 0))
   )
+  (wire (pts (xy 184.15 132.08) (xy 187.96 132.08))
+    (stroke (width 0) (type default) (color 0 0 0 0))
+  )
+  (wire (pts (xy 72.39 35.56) (xy 63.5 35.56))
+    (stroke (width 0) (type default) (color 0 0 0 0))
+  )
   (wire (pts (xy 87.63 149.86) (xy 93.98 149.86))
     (stroke (width 0) (type default) (color 0 0 0 0))
@@
     (stroke (width 0) (type default) (color 0 0 0 0))
   )
+  (wire (pts (xy 184.15 127) (xy 187.96 127))
+    (stroke (width 0) (type default) (color 0 0 0 0))
+  )
   (wire (pts (xy 63.5 69.85) (xy 63.5 73.66))
     (stroke (width 0) (type default) (color 0 0 0 0))
@@
     (stroke (width 0) (type default) (color 0 0 0 0))
   )
-  (wire (pts (xy 179.07 127) (xy 187.96 127))
+  (wire (pts (xy 63.5 35.56) (xy 63.5 39.37))
     (stroke (width 0) (type default) (color 0 0 0 0))
   )
@@
     (stroke (width 0) (type default) (color 0 0 0 0))
   )
-  (wire (pts (xy 182.88 110.49) (xy 182.88 114.3))
+  (wire (pts (xy 182.88 110.49) (xy 182.88 111.76))
     (stroke (width 0) (type default) (color 0 0 0 0))
   )
@@
     (stroke (width 0) (type default) (color 0 0 0 0))
   )
+  (wire (pts (xy 179.07 129.54) (xy 187.96 129.54))
+    (stroke (width 0) (type default) (color 0 0 0 0))
+  )
   (wire (pts (xy 87.63 147.32) (xy 93.98 147.32))
     (stroke (width 0) (type default) (color 0 0 0 0))
@@
     (stroke (width 0) (type default) (color 0 0 0 0))
   )
-  (wire (pts (xy 63.5 33.02) (xy 63.5 36.83))
+  (wire (pts (xy 184.15 134.62) (xy 184.15 132.08))
+    (stroke (width 0) (type default) (color 0 0 0 0))
+  )
+  (wire (pts (xy 63.5 33.02) (xy 63.5 35.56))
     (stroke (width 0) (type default) (color 0 0 0 0))
   )
@@
     (stroke (width 0) (type default) (color 0 0 0 0))
   )
-  (text "speaker" (at 191.77 118.11 180)
+  (wire (pts (xy 59.69 39.37) (xy 63.5 39.37))
+    (stroke (width 0) (type default) (color 0 0 0 0))
+  )
+  (text "speaker" (at 194.31 121.92 180)
     (effects (font (size 1.27 1.27)) (justify right bottom))
   )
@@
     )
   )
+  (global_label "MIDI_IN_GND" (shape input) (at 59.69 39.37 180) (fields_autoplaced)
+    (effects (font (size 1.27 1.27)) (justify right))
+    (property "Intersheet References" "${INTERSHEET_REFS}" (id 0) (at 45.605 39.2906 0)
+      (effects (font (size 1.27 1.27)) (justify right) hide)
+    )
+  )
   (global_label "MIDI_THRU" (shape input) (at 36.83 64.77 180) (fields_autoplaced)
     (effects (font (size 1.27 1.27)) (justify right))
@@
     )
   )
-  (global_label "SOUTL" (shape input) (at 179.07 127 180) (fields_autoplaced)
-    (effects (font (size 1.27 1.27)) (justify right))
-    (property "Intersheet References" "${INTERSHEET_REFS}" (id 0) (at 170.7907 126.9206 0)
+  (global_label "SOUTL" (shape input) (at 179.07 129.54 180) (fields_autoplaced)
+    (effects (font (size 1.27 1.27)) (justify right))
+    (property "Intersheet References" "${INTERSHEET_REFS}" (id 0) (at 170.7907 129.4606 0)
       (effects (font (size 1.27 1.27)) (justify right) hide)
     )
@@
     (pin "9")
   )
-  (symbol (lib_id "power:GND") (at 63.5 36.83 0) (unit 1)
-    (in_bom yes) (on_board yes) (fields_autoplaced)
-    (property "Reference" "#PWR013" (id 0) (at 63.5 43.18 0)
-      (effects (font (size 1.27 1.27)) hide)
-    )
-    (property "Value" "GND" (id 1) (at 63.5 41.91 0))
-    (property "Footprint" "" (id 2) (at 63.5 36.83 0)
-      (effects (font (size 1.27 1.27)) hide)
-    )
-    (property "Datasheet" "" (id 3) (at 63.5 36.83 0)
-      (effects (font (size 1.27 1.27)) hide)
-    )
-    (pin "1")
-  )
-  (symbol (lib_id "power:GND") (at 72.39 33.02 0) (unit 1)
-    (in_bom yes) (on_board yes) (fields_autoplaced)
-    (property "Reference" "#PWR015" (id 0) (at 72.39 39.37 0)
-      (effects (font (size 1.27 1.27)) hide)
-    )
-    (property "Value" "GND" (id 1) (at 72.39 38.1 0))
-    (property "Footprint" "" (id 2) (at 72.39 33.02 0)
-      (effects (font (size 1.27 1.27)) hide)
-    )
-    (property "Datasheet" "" (id 3) (at 72.39 33.02 0)
-      (effects (font (size 1.27 1.27)) hide)
-    )
-    (pin "1")
-  )
-  (symbol (lib_id "Connector:Conn_01x02_Male") (at 193.04 127 180) (unit 1)
-    (in_bom yes) (on_board yes) (fields_autoplaced)
-    (property "Reference" "J8" (id 0) (at 192.405 132.08 0))
-    (property "Value" "Conn_01x02_Male" (id 1) (at 192.405 129.54 0))
-    (property "Footprint" "Capacitor_THT:C_Rect_L7.5mm_W6.5mm_P5.00mm" (id 2) (at 193.04 127 0)
-      (effects (font (size 1.27 1.27)) hide)
-    )
-    (property "Datasheet" "~" (id 3) (at 193.04 127 0)
-      (effects (font (size 1.27 1.27)) hide)
-    )
-    (pin "1")
-    (pin "2")
-  )
   (symbol (lib_id "Device:R") (at 44.45 101.6 90) (unit 1)
     (in_bom yes) (on_board yes) (fields_autoplaced)
@@
     (pin "1")
   )
+  (symbol (lib_id "Connector:Conn_01x04_Male") (at 193.04 129.54 180) (unit 1)
+    (in_bom yes) (on_board yes) (fields_autoplaced)
+    (property "Reference" "J6" (id 0) (at 194.31 126.9999 0)
+      (effects (font (size 1.27 1.27)) (justify right))
+    )
+    (property "Value" "Conn_01x04_Male" (id 1) (at 194.31 129.5399 0)
+      (effects (font (size 1.27 1.27)) (justify right))
+    )
+    (property "Footprint" "Connector_PinHeader_2.54mm:PinHeader_1x04_P2.54mm_Vertical" (id 2) (at 193.04 129.54 0)
+      (effects (font (size 1.27 1.27)) hide)
+    )
+    (property "Datasheet" "~" (id 3) (at 193.04 129.54 0)
+      (effects (font (size 1.27 1.27)) hide)
+    )
+    (pin "1")
+    (pin "2")
+    (pin "3")
+    (pin "4")
+  )
   (symbol (lib_id "power:+5V") (at 205.74 45.72 0) (unit 1)
     (in_bom yes) (on_board yes) (fields_autoplaced)
@@
     (pin "1")
   )
-  (symbol (lib_id "power:GND") (at 182.88 114.3 0) (unit 1)
-    (in_bom yes) (on_board yes) (fields_autoplaced)
-    (property "Reference" "#PWR045" (id 0) (at 182.88 120.65 0)
-      (effects (font (size 1.27 1.27)) hide)
-    )
-    (property "Value" "GND" (id 1) (at 182.88 119.38 0))
-    (property "Footprint" "" (id 2) (at 182.88 114.3 0)
-      (effects (font (size 1.27 1.27)) hide)
-    )
-    (property "Datasheet" "" (id 3) (at 182.88 114.3 0)
+  (symbol (lib_id "power:GND") (at 182.88 111.76 0) (unit 1)
+    (in_bom yes) (on_board yes) (fields_autoplaced)
+    (property "Reference" "#PWR045" (id 0) (at 182.88 118.11 0)
+      (effects (font (size 1.27 1.27)) hide)
+    )
+    (property "Value" "GND" (id 1) (at 182.88 116.84 0))
+    (property "Footprint" "" (id 2) (at 182.88 111.76 0)
+      (effects (font (size 1.27 1.27)) hide)
+    )
+    (property "Datasheet" "" (id 3) (at 182.88 111.76 0)
       (effects (font (size 1.27 1.27)) hide)
     )
@@
     (pin "2")
   )
+  (symbol (lib_id "power:GND") (at 184.15 134.62 0) (unit 1)
+    (in_bom yes) (on_board yes) (fields_autoplaced)
+    (property "Reference" "#PWR0107" (id 0) (at 184.15 140.97 0)
+      (effects (font (size 1.27 1.27)) hide)
+    )
+    (property "Value" "GND" (id 1) (at 184.15 139.7 0))
+    (property "Footprint" "" (id 2) (at 184.15 134.62 0)
+      (effects (font (size 1.27 1.27)) hide)
+    )
+    (property "Datasheet" "" (id 3) (at 184.15 134.62 0)
+      (effects (font (size 1.27 1.27)) hide)
+    )
+    (pin "1")
+  )
   (symbol (lib_id "Device:C") (at 259.08 45.72 0) (unit 1)

Commit message: gerber files generated
Connections:
- net GND: now also U11.11 (5A), U11.13 (6A)
Changed lines of the file:
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@@
   (junction (at 214.63 53.34) (diameter 0) (color 0 0 0 0)
   )
+  (junction (at 49.53 154.94) (diameter 0) (color 0 0 0 0)
+  )
   (junction (at 171.45 50.8) (diameter 0) (color 0 0 0 0)
   )
@@
     (stroke (width 0) (type default) (color 0 0 0 0))
   )
+  (wire (pts (xy 49.53 161.29) (xy 49.53 154.94))
+    (stroke (width 0) (type default) (color 0 0 0 0))
+  )
   (wire (pts (xy 181.61 60.96) (xy 181.61 58.42))
     (stroke (width 0) (type default) (color 0 0 0 0))
@@
     (stroke (width 0) (type default) (color 0 0 0 0))
   )
+  (wire (pts (xy 49.53 152.4) (xy 52.07 152.4))
+    (stroke (width 0) (type default) (color 0 0 0 0))
+  )
   (wire (pts (xy 87.63 160.02) (xy 91.44 160.02))
     (stroke (width 0) (type default) (color 0 0 0 0))
@@
     (stroke (width 0) (type default) (color 0 0 0 0))
   )
+  (wire (pts (xy 49.53 154.94) (xy 49.53 152.4))
+    (stroke (width 0) (type default) (color 0 0 0 0))
+  )
   (wire (pts (xy 259.08 49.53) (xy 259.08 50.8))
     (stroke (width 0) (type default) (color 0 0 0 0))
@@
   )
   (wire (pts (xy 196.85 50.8) (xy 200.66 50.8))
+    (stroke (width 0) (type default) (color 0 0 0 0))
+  )
+  (wire (pts (xy 49.53 154.94) (xy 52.07 154.94))
     (stroke (width 0) (type default) (color 0 0 0 0))
   )
@@
     (pin "2")
   )
+  (symbol (lib_id "power:GND") (at 49.53 161.29 0) (unit 1)
+    (in_bom yes) (on_board yes) (fields_autoplaced)
+    (property "Reference" "#PWR07" (id 0) (at 49.53 167.64 0)
+      (effects (font (size 1.27 1.27)) hide)
+    )
+    (property "Value" "GND" (id 1) (at 49.53 166.37 0))
+    (property "Footprint" "" (id 2) (at 49.53 161.29 0)
+      (effects (font (size 1.27 1.27)) hide)
+    )
+    (property "Datasheet" "" (id 3) (at 49.53 161.29 0)
+      (effects (font (size 1.27 1.27)) hide)
+    )
+    (pin "1")
+  )
   (symbol (lib_id "power:GND") (at 91.44 161.29 0) (unit 1)
